Commit message: 3-16 modify configuration file

File: src/collaborative-robotic-sanding/fanuc_r2000ic_support/urdf/r2000ic165f.xacro (robot description, xacro)
@@ -1,4 +1,4 @@
 <?xml version="1.0" encoding="utf-8" ?>
-<robot name="fanuc_r2000ic165f" xmlns:xacro="http://wiki.ros.org/xacro">
+<robot name="crs" xmlns:xacro="http://wiki.ros.org/xacro">
   <xacro:include filename="$(find fanuc_r2000ic_support)/urdf/r2000ic165f_macro.xacro"/>
   <xacro:fanuc_r2000ic165f prefix=""/>

File: src/collaborative-robotic-sanding/fanuc_r2000ic_support/urdf/r2000ic165f_macro.xacro (robot description, xacro)
@@ -173,6 +173,5 @@
       <limit lower="${radians(-360)}" upper="${radians(360)}" effort="0" velocity="${radians(260)}"/>
     </joint>
-<!--
-<link name="part_link">
+<!--<link name="part_link">
   <visual>
     <origin xyz="0 0 0" rpy="0 0 0"/>
@@ -216,121 +215,158 @@
           <child link="${prefix}ef" />
         </joint>
-<transmission name="joint_1">
-    <type>transmission_interface/SimpleTransmission</type>
-    <joint name="joint_1">
-        <hardwareInterface>hardware_interface/EffortJointInterface</hardwareInterface>
-    </joint>
-    <actuator name="joint_1_motor">
-        <hardwareInterface>hardware_interface/EffortJointInterface</hardwareInterface>
-        <mechanicalReduction>1</mechanicalReduction>
-    </actuator>
-</transmission>
-<gazebo reference="base_link">
-    <selfCollide>true</selfCollide>
-</gazebo>
-<gazebo reference="link_1">
-    <selfCollide>true</selfCollide>
-</gazebo>
-<gazebo reference="link_2">
-    <selfCollide>true</selfCollide>
-</gazebo>
-<gazebo reference="link_3">
-    <selfCollide>true</selfCollide>
-</gazebo>
-<gazebo reference="link_4">
-    <selfCollide>true</selfCollide>
-</gazebo>
-<gazebo reference="link_5">
-    <selfCollide>true</selfCollide>
-</gazebo>
-<gazebo reference="link_6">
-    <selfCollide>true</selfCollide>
-</gazebo>
-<gazebo reference="joint_1">
-    <selfCollide>true</selfCollide>
-</gazebo>
-<gazebo reference="joint_2">
-    <selfCollide>true</selfCollide>
-</gazebo>
-<gazebo reference="joint_3">
-    <selfCollide>true</selfCollide>
-</gazebo>
-<gazebo reference="base">
-    <selfCollide>true</selfCollide>
-</gazebo>
-<gazebo reference="flange">
-    <selfCollide>true</selfCollide>
-</gazebo>
-<gazebo reference="tool0">
-    <selfCollide>true</selfCollide>
-</gazebo>
-<gazebo reference="gazebo_camera_link">
-    <sensor type="depth" name="sensor_name">
-      <!-- Set always_on only sensor, not on plugin -->
-      <always_on>1</always_on>
-      <!-- Set update_rate only sensor, not on plugin -->
-      <update_rate>5</update_rate>
-      <camera name="camera_name">
-        <image>
-          <width>320</width>
-          <height>200</height>
-        </image>
-        <distortion>
-          <k1>-0.0</k1>
-          <k2>0.0</k2>
-          <k3>0.0</k3>
-          <p1>-0.0</p1>
-          <p2>-0.0</p2>
-          <center>0.5 0.5</center>
-        </distortion>
-      </camera>
-      <plugin name="plugin_name" filename="libgazebo_ros_camera.so">
-        <!-- Change namespace, camera name and topics so:
-             * Raw images are published to: /custom_ns/custom_camera/custom_image
-             * Depth images are published to: /custom_ns/custom_camera/custom_image_depth
-             * Raw image camera info is published to: /custom_ns/custom_camera/custom_info_raw
-             * Depth image camera info is published to: /custom_ns/custom_camera/custom_info_depth
-             * Point cloud is published to: /custom_ns/custom_camera/custom_points
-        -->
-        <ros>
-          <namespace>custom_ns</namespace>
-          <argument>camera/image_raw:=camera/custom_image</argument>
-          <argument>camera/image_depth:=camera/custom_image_depth</argument>
-          <argument>camera/camera_info:=camera/custom_info_raw</argument>
-          <argument>camera/camera_info_depth:=camera/custom_info_depth</argument>
-          <argument>camera/points:=camera/pointcloud</argument>
-        </ros>
-        <!-- Set camera name. If empty, defaults to sensor name (i.e. "sensor_name") -->
-        <camera_name>camera</camera_name>
-        <frame_name>camera_link_optical</frame_name>
-        <!-- Set TF frame name. If empty, defaults to link name (i.e. "link_name") -->
-        <hack_baseline>0.07</hack_baseline>
-        <!-- No need to repeat distortion parameters or to set autoDistortion -->
-         <min_depth>0.1</min_depth>
-      </plugin>
-    </sensor>
-</gazebo>
-<gazebo>
-    <plugin name='gazebo_ros_joint_state_publisher' filename='libgazebo_ros_joint_state_publisher.so'>
-      <ros>
-          <namespace>/test</namespace>
-          <argument>joint_states:=joint_states</argument>
-      </ros>
-      <update_rate>50</update_rate>
-      <joint_name>joint_1</joint_name>
-      <joint_name>joint_2</joint_name>
-      <joint_name>joint_3</joint_name>
-      <joint_name>joint_4</joint_name>
-      <joint_name>joint_5</joint_name>
-      <joint_name>joint_6</joint_name>
-    </plugin>
-    <plugin name='crs_gazebo_plugins_joint_pose_trajectory' filename='libcrs_gazebo_plugins_joint_pose_trajectory.so'>
-        <ros>
-          <namespace>sim</namespace>
-          <argument>follow_joint_trajectory:=follow_joint_trajectory</argument>
-        </ros>
-        <update_rate>20</update_rate>
-    </plugin>
-</gazebo>
+    <link name="${prefix}gazebo_camera_link" />
+    <joint name="${prefix}gazebo_camera_joint" type="fixed">
+        <origin xyz="0.0 0.0 0.0" rpy="1.57 -1.57 0.0"/>
+        <parent link="${prefix}camera_link_optical"/>
+        <child link="${prefix}gazebo_camera_link"/>
+    </joint>
+    <link name="${prefix}camera_link_optical" />
+    <joint name="${prefix}camera_optical_joint" type="fixed">
+        <origin xyz="-0.021 0.0797 0.06525" rpy="-0.7854 0 0"/>
+        <parent link="${prefix}ef"/>
+        <child link="${prefix}camera_link_optical"/>
+    </joint>
+    <link name="${prefix}camera_link" />
+    <joint name="${prefix}camera_link_joint" type="fixed">
+        <origin xyz="0.0 0.0 0.0" rpy="1.57 -1.57 0"/>
+        <parent link="${prefix}camera_link_optical"/>
+        <child link="${prefix}camera_link"/>
+    </joint>
+    <transmission name="joint_1">
+        <type>transmission_interface/SimpleTransmission</type>
+        <joint name="joint_1">
+            <hardwareInterface>hardware_interface/EffortJointInterface</hardwareInterface>
+        </joint>
+        <actuator name="joint_1_motor">
+            <hardwareInterface>hardware_interface/EffortJointInterface</hardwareInterface>
+            <mechanicalReduction>1</mechanicalReduction>
+        </actuator>
+    </transmission>
+    <gazebo reference="${prefix}base_link">
+        <selfCollide>true</selfCollide>
+    </gazebo>
+    <gazebo reference="${prefix}link_1">
+        <selfCollide>true</selfCollide>
+    </gazebo>
+    <gazebo reference="${prefix}link_2">
+        <selfCollide>true</selfCollide>
+    </gazebo>
+    <gazebo reference="${prefix}link_3">
+        <selfCollide>true</selfCollide>
+    </gazebo>
+    <gazebo reference="${prefix}link_4">
+        <selfCollide>true</selfCollide>
+    </gazebo>
+    <gazebo reference="${prefix}link_5">
+        <selfCollide>true</selfCollide>
+    </gazebo>
+    <gazebo reference="${prefix}link_6">
+        <selfCollide>true</selfCollide>
+    </gazebo>
+    <gazebo reference="${prefix}ef">
+        <selfCollide>true</selfCollide>
+    </gazebo>
+    <gazebo reference="${prefix}joint_1">
+        <selfCollide>true</selfCollide>
+    </gazebo>
+    <gazebo reference="${prefix}joint_2">
+        <selfCollide>true</selfCollide>
+    </gazebo>
+    <gazebo reference="${prefix}joint_3">
+        <selfCollide>true</selfCollide>
+    </gazebo>
+    <gazebo reference="${prefix}joint_4">
+        <selfCollide>true</selfCollide>
+    </gazebo>
+    <gazebo reference="${prefix}joint_5">
+        <selfCollide>true</selfCollide>
+    </gazebo>
+    <gazebo reference="${prefix}joint_6">
+        <selfCollide>true</selfCollide>
+    </gazebo>
+    <gazebo reference="${prefix}flange-ef">
+        <selfCollide>true</selfCollide>
+    </gazebo>
+    <gazebo reference="${prefix}tool0">
+        <selfCollide>true</selfCollide>
+    </gazebo>
+    <gazebo reference="${prefix}base">
+        <selfCollide>true</selfCollide>
+    </gazebo>
+    <gazebo reference="${prefix}flange">
+        <selfCollide>true</selfCollide>
+    </gazebo>
+    <gazebo reference="tool0">
+        <selfCollide>true</selfCollide>
+    </gazebo>
+    <gazebo reference="gazebo_camera_link">
+        <sensor type="depth" name="sensor_name">
+          <!-- Set always_on only sensor, not on plugin -->
+          <always_on>1</always_on>
+          <!-- Set update_rate only sensor, not on plugin -->
+          <update_rate>5</update_rate>
+          <camera name="camera_name">
+            <image>
+              <width>320</width>
+              <height>200</height>
+            </image>
+            <distortion>
+              <k1>-0.0</k1>
+              <k2>0.0</k2>
+              <k3>0.0</k3>
+              <p1>-0.0</p1>
+              <p2>-0.0</p2>
+              <center>0.5 0.5</center>
+            </distortion>
+          </camera>
+          <plugin name="plugin_name" filename="libgazebo_ros_camera.so">
+            <!-- Change namespace, camera name and topics so:
+                 * Raw images are published to: /custom_ns/custom_camera/custom_image
+                 * Depth images are published to: /custom_ns/custom_camera/custom_image_depth
+                 * Raw image camera info is published to: /custom_ns/custom_camera/custom_info_raw
+                 * Depth image camera info is published to: /custom_ns/custom_camera/custom_info_depth
+                 * Point cloud is published to: /custom_ns/custom_camera/custom_points
+            -->
+            <ros>
+              <namespace>custom_ns</namespace>
+              <argument>camera/image_raw:=camera/custom_image</argument>
+              <argument>camera/image_depth:=camera/custom_image_depth</argument>
+              <argument>camera/camera_info:=camera/custom_info_raw</argument>
+              <argument>camera/camera_info_depth:=camera/custom_info_depth</argument>
+              <argument>camera/points:=camera/pointcloud</argument>
+            </ros>
+            <!-- Set camera name. If empty, defaults to sensor name (i.e. "sensor_name") -->
+            <camera_name>camera</camera_name>
+            <frame_name>camera_link_optical</frame_name>
+            <!-- Set TF frame name. If empty, defaults to link name (i.e. "link_name") -->
+            <hack_baseline>0.07</hack_baseline>
+            <!-- No need to repeat distortion parameters or to set autoDistortion -->
+             <min_depth>0.1</min_depth>
+          </plugin>
+        </sensor>
+    </gazebo>
+    <gazebo>
+        <plugin name='gazebo_ros_joint_state_publisher' filename='libgazebo_ros_joint_state_publisher.so'>
+          <ros>
+              <namespace>/crs</namespace>
+              <argument>joint_states:=joint_states</argument>
+          </ros>
+          <update_rate>50</update_rate>
+          <joint_name>${prefix}joint_1</joint_name>
+          <joint_name>${prefix}joint_2</joint_name>
+          <joint_name>${prefix}joint_3</joint_name>
+          <joint_name>${prefix}joint_4</joint_name>
+          <joint_name>${prefix}joint_5</joint_name>
+          <joint_name>${prefix}joint_6</joint_name>
+          <joint_name>${prefix}flange-ef</joint_name>
+        </plugin>
+        <plugin name='crs_gazebo_plugins_joint_pose_trajectory' filename='libcrs_gazebo_plugins_joint_pose_trajectory.so'>
+            <ros>
+              <namespace>sim</namespace>
+              <argument>follow_joint_trajectory:=follow_joint_trajectory</argument>
+            </ros>
+            <update_rate>20</update_rate>
+        </plugin>
+    </gazebo>
   </xacro:macro>
 </robot>
