Commit message: 3-3 apppanel+fanuc

File: src/collaborative-robotic-sanding/fanuc_r2000ic_support/urdf/r2000ic165f_macro.xacro (robot description, xacro)
@@ -4,4 +4,10 @@
   <xacro:macro name="fanuc_r2000ic165f" params="prefix">
     <!-- links: main serial chain -->
+    <link name="world" />
+    <joint name="${prefix}world_base_link" type="fixed">
+        <parent link="world" />
+        <child link="${prefix}base_link" />
+        <origin rpy="0 0 0" xyz="-2.5 0 0" />
+    </joint>
     <link name="${prefix}base_link">
       <visual>
@@ -173,4 +179,121 @@
       <child link="${prefix}tool0" />
     </joint>
+<transmission name="joint_1">
+    <type>transmission_interface/SimpleTransmission</type>
+    <joint name="${prefix}joint_1">
+        <hardwareInterface>hardware_interface/EffortJointInterface</hardwareInterface>
+    </joint>
+    <actuator name="joint_1_motor">
+        <hardwareInterface>hardware_interface/EffortJointInterface</hardwareInterface>
+        <mechanicalReduction>1</mechanicalReduction>
+    </actuator>
+</transmission>
+<gazebo reference="${prefix}base_link">
+    <selfCollide>true</selfCollide>
+</gazebo>
+<gazebo reference="${prefix}link_1">
+    <selfCollide>true</selfCollide>
+</gazebo>
+<gazebo reference="${prefix}link_2">
+    <selfCollide>true</selfCollide>
+</gazebo>
+<gazebo reference="${prefix}link_3">
+    <selfCollide>true</selfCollide>
+</gazebo>
+<gazebo reference="${prefix}link_4">
+    <selfCollide>true</selfCollide>
+</gazebo>
+<gazebo reference="${prefix}link_5">
+    <selfCollide>true</selfCollide>
+</gazebo>
+<gazebo reference="${prefix}link_6">
+    <selfCollide>true</selfCollide>
+</gazebo>
+<gazebo reference="${prefix}joint_1">
+    <selfCollide>true</selfCollide>
+</gazebo>
+<gazebo reference="${prefix}joint_2">
+    <selfCollide>true</selfCollide>
+</gazebo>
+<gazebo reference="${prefix}joint_3">
+    <selfCollide>true</selfCollide>
+</gazebo>
+<gazebo reference="${prefix}base">
+    <selfCollide>true</selfCollide>
+</gazebo>
+<gazebo reference="${prefix}flange">
+    <selfCollide>true</selfCollide>
+</gazebo>
+<gazebo reference="${prefix}tool0">
+    <selfCollide>true</selfCollide>
+</gazebo>
+<gazebo reference="${prefix}gazebo_camera_link">
+    <sensor type="depth" name="sensor_name">
+      <!-- Set always_on only sensor, not on plugin -->
+      <always_on>1</always_on>
+      <!-- Set update_rate only sensor, not on plugin -->
+      <update_rate>5</update_rate>
+      <camera name="camera_name">
+        <image>
+          <width>320</width>
+          <height>200</height>
+        </image>
+        <distortion>
+          <k1>-0.0</k1>
+          <k2>0.0</k2>
+          <k3>0.0</k3>
+          <p1>-0.0</p1>
+          <p2>-0.0</p2>
+          <center>0.5 0.5</center>
+        </distortion>
+      </camera>
+      <plugin name="plugin_name" filename="libgazebo_ros_camera.so">
+        <!-- Change namespace, camera name and topics so:
+             * Raw images are published to: /custom_ns/custom_camera/custom_image
+             * Depth images are published to: /custom_ns/custom_camera/custom_image_depth
+             * Raw image camera info is published to: /custom_ns/custom_camera/custom_info_raw
+             * Depth image camera info is published to: /custom_ns/custom_camera/custom_info_depth
+             * Point cloud is published to: /custom_ns/custom_camera/custom_points
+        -->
+        <ros>
+          <namespace>custom_ns</namespace>
+          <argument>camera/image_raw:=camera/custom_image</argument>
+          <argument>camera/image_depth:=camera/custom_image_depth</argument>
+          <argument>camera/camera_info:=camera/custom_info_raw</argument>
+          <argument>camera/camera_info_depth:=camera/custom_info_depth</argument>
+          <argument>camera/points:=camera/pointcloud</argument>
+        </ros>
+        <!-- Set camera name. If empty, defaults to sensor name (i.e. "sensor_name") -->
+        <camera_name>camera</camera_name>
+        <frame_name>camera_link_optical</frame_name>
+        <!-- Set TF frame name. If empty, defaults to link name (i.e. "link_name") -->
+        <hack_baseline>0.07</hack_baseline>
+        <!-- No need to repeat distortion parameters or to set autoDistortion -->
+         <min_depth>0.1</min_depth>
+      </plugin>
+    </sensor>
+</gazebo>
+<gazebo>
+    <plugin name='gazebo_ros_joint_state_publisher' filename='libgazebo_ros_joint_state_publisher.so'>
+      <ros>
+          <namespace>/test</namespace>
+          <argument>joint_states:=joint_states</argument>
+      </ros>
+      <update_rate>50</update_rate>
+      <joint_name>${prefix}joint_1</joint_name>
+      <joint_name>${prefix}joint_2</joint_name>
+      <joint_name>${prefix}joint_3</joint_name>
+      <joint_name>${prefix}joint_4</joint_name>
+      <joint_name>${prefix}joint_5</joint_name>
+      <joint_name>${prefix}joint_6</joint_name>
+    </plugin>
+    <plugin name='crs_gazebo_plugins_joint_pose_trajectory' filename='libcrs_gazebo_plugins_joint_pose_trajectory.so'>
+        <ros>
+          <namespace>sim</namespace>
+          <argument>follow_joint_trajectory:=${prefix}follow_joint_trajectory</argument>
+        </ros>
+        <update_rate>20</update_rate>
+    </plugin>
+</gazebo>
   </xacro:macro>
 </robot>

Commit message: 3-12 modify motion plan

File: src/collaborative-robotic-sanding/fanuc_r2000ic_support/urdf/r2000ic165f_macro.xacro (robot description, xacro)
@@ -158,4 +158,20 @@
       <limit lower="${radians(-360)}" upper="${radians(360)}" effort="0" velocity="${radians(260)}"/>
     </joint>
+<link name="part_link">
+  <visual>
+    <origin xyz="0 0 0" rpy="0 0 0"/>
+    <geometry>
+      <mesh filename="package://fanuc_r2000ic_support/meshes/r2000ic165f/visual/sandpart.stl"/>
+    </geometry>
+    <material name="">
+      <color rgba="0.9 0.7 0.4 1.0"/>
+    </material>
+  </visual>
+</link>
+  <joint name="world_part_link" type="fixed">
+      <parent link="base_link" />
+      <child link="part_link" />
+      <origin rpy="0 0 0" xyz="1.4 -0.4 0.6" />
+  </joint>
     <!-- ROS-Industrial 'base' frame: base_link to Fanuc World Coordinates transform -->
     <link name="${prefix}base" />

Commit message: 3-26 add generate_baselink

File: src/collaborative-robotic-sanding/fanuc_r2000ic_support/urdf/r2000ic165f_macro.xacro (robot description, xacro)
@@ -235,5 +235,5 @@
     <transmission name="joint_1">
         <type>transmission_interface/SimpleTransmission</type>
-        <joint name="joint_1">
+        <joint name="${prefix}joint_1">
             <hardwareInterface>hardware_interface/EffortJointInterface</hardwareInterface>
         </joint>
@@ -243,4 +243,54 @@
         </actuator>
     </transmission>
+<transmission name="joint_2">
+    <type>transmission_interface/SimpleTransmission</type>
+    <joint name="${prefix}joint_2">
+        <hardwareInterface>hardware_interface/EffortJointInterface</hardwareInterface>
+    </joint>
+    <actuator name="joint_2_motor">
+        <hardwareInterface>hardware_interface/EffortJointInterface</hardwareInterface>
+        <mechanicalReduction>1</mechanicalReduction>
+    </actuator>
+</transmission>
+<transmission name="joint_3">
+    <type>transmission_interface/SimpleTransmission</type>
+    <joint name="${prefix}joint_3">
+        <hardwareInterface>hardware_interface/EffortJointInterface</hardwareInterface>
+    </joint>
+    <actuator name="joint_3_motor">
+        <hardwareInterface>hardware_interface/EffortJointInterface</hardwareInterface>
+        <mechanicalReduction>1</mechanicalReduction>
+    </actuator>
+</transmission>
+<transmission name="joint_4">
+    <type>transmission_interface/SimpleTransmission</type>
+    <joint name="${prefix}joint_4">
+        <hardwareInterface>hardware_interface/EffortJointInterface</hardwareInterface>
+    </joint>
+    <actuator name="joint_4_motor">
+        <hardwareInterface>hardware_interface/EffortJointInterface</hardwareInterface>
+        <mechanicalReduction>1</mechanicalReduction>
+    </actuator>
+</transmission>
+<transmission name="joint_5">
+    <type>transmission_interface/SimpleTransmission</type>
+    <joint name="${prefix}joint_5">
+        <hardwareInterface>hardware_interface/EffortJointInterface</hardwareInterface>
+    </joint>
+    <actuator name="joint_5_motor">
+        <hardwareInterface>hardware_interface/EffortJointInterface</hardwareInterface>
+        <mechanicalReduction>1</mechanicalReduction>
+    </actuator>
+</transmission>
+<transmission name="joint_6">
+    <type>transmission_interface/SimpleTransmission</type>
+    <joint name="${prefix}joint_6">
+        <hardwareInterface>hardware_interface/EffortJointInterface</hardwareInterface>
+    </joint>
+    <actuator name="joint_6_motor">
+        <hardwareInterface>hardware_interface/EffortJointInterface</hardwareInterface>
+        <mechanicalReduction>1</mechanicalReduction>
+    </actuator>
+</transmission>
     <gazebo reference="${prefix}base_link">
         <selfCollide>true</selfCollide>

Commit message: 2021 3-29 add gazebo inertial tag

File: src/collaborative-robotic-sanding/fanuc_r2000ic_support/urdf/r2000ic165f_macro.xacro (robot description, xacro)
@@ -24,4 +24,9 @@
         </geometry>
       </collision>
+      <inertial>
+          <mass value="10.0" />
+          <origin rpy="0 0 0" xyz="0.0 0.0 0.0" />
+          <inertia ixx="0.002695" ixy="0.000023" ixz="0.000157" iyy="0.004043" iyz="0.000023" izz="0.006096" />
+      </inertial>
     </link>
     <link name="${prefix}link_1">
@@ -39,4 +44,9 @@
         </geometry>
       </collision>
+      <inertial>
+          <mass value="4.0" />
+          <origin rpy="0 0 0" xyz="0.0 0.0 0.0" />
+          <inertia ixx="0.012932" ixy="0.003309" ixz=" -0.000331" iyy="0.018366" iyz="-0.000071" izz="0.019767" />
+      </inertial>
     </link>
     <link name="${prefix}link_2">
@@ -54,4 +64,9 @@
         </geometry>
       </collision>
+      <inertial>
+          <mass value="3.0" />
+          <origin rpy="0 0 0" xyz="0.0 0.0 0.0" />
+          <inertia ixx="0.014390" ixy="0.000091" ixz="-0.000323" iyy="0.015120" iyz="-0.001213" izz="0.002053" />
+      </inertial>
     </link>
     <link name="${prefix}link_3">
@@ -69,4 +84,9 @@
         </geometry>
       </collision>
+      <inertial>
+          <mass value="5.0" />
+          <origin rpy="0 0 0" xyz="0.0 0.0 0.0" />
+          <inertia ixx="0.001451" ixy="0.000017" ixz="-0.000177" iyy="0.001441" iyz="0.000072" izz="0.001041" />
+      </inertial>
     </link>
     <link name="${prefix}link_4">
@@ -84,4 +104,9 @@
         </geometry>
       </collision>
+      <inertial>
+          <mass value="5.0" />
+          <origin rpy="0 0 0" xyz="0.0 0.0 0.0" />
+          <inertia ixx="0.000333" ixy="0.000044" ixz="0.000006" iyy="0.004287" iyz="-0.000000" izz="0.004282" />
+      </inertial>
     </link>
     <link name="${prefix}link_5">
@@ -99,4 +124,9 @@
         </geometry>
       </collision>
+      <inertial>
+          <mass value="5.0" />
+          <origin rpy="0 0 0" xyz="0.0 0.0 0.0" />
+          <inertia ixx="0.000088" ixy="-0.000012" ixz="0.000000" iyy="0.000094" iyz="0.000000" izz="0.000118" />
+      </inertial>
     </link>
     <link name="${prefix}link_6">
@@ -114,4 +144,9 @@
         </geometry>
       </collision>
+      <inertial>
+          <mass value="7.0" />
+          <origin rpy="0 0 0" xyz="0.0 0.0 0.0" />
+          <inertia ixx="0.000002" ixy="0.000000" ixz="-0.000000" iyy="0.000001" iyz="0.000000" izz="0.000001" />
+      </inertial>
     </link>
     <link name="${prefix}ef">
@@ -129,4 +164,9 @@
             </geometry>
           </collision>
+          <inertial>
+              <mass value="3.0" />
+              <origin rpy="0 0 0" xyz="0.0 0.0 0.0" />
+              <inertia ixx="0.000127" ixy="0.000000" ixz="0.000052" iyy="0.000194" iyz="0.000003" izz="0.000141" />
+          </inertial>
         </link>
     <!-- joints: main serial chain -->
@@ -399,5 +439,5 @@
         <plugin name='gazebo_ros_joint_state_publisher' filename='libgazebo_ros_joint_state_publisher.so'>
           <ros>
-              <namespace>/crs</namespace>
+              <namespace>/test</namespace>
               <argument>joint_states:=joint_states</argument>
           </ros>
@@ -409,5 +449,4 @@
           <joint_name>${prefix}joint_5</joint_name>
           <joint_name>${prefix}joint_6</joint_name>
-          <joint_name>${prefix}flange-ef</joint_name>
         </plugin>
         <plugin name='crs_gazebo_plugins_joint_pose_trajectory' filename='libcrs_gazebo_plugins_joint_pose_trajectory.so'>

Commit message: 2021-4-1 add generate ls file

File: src/collaborative-robotic-sanding/fanuc_r2000ic_support/urdf/r2000ic165f_macro.xacro (robot description, xacro)
@@ -24,4 +24,9 @@
         </geometry>
       </collision>
+      <!--
+      <inertial>
+               <mass value="0.0" />
+                <inertia ixx="0.002695" ixy="0.000023" ixz="0.000157" iyy="0.004043" iyz="0.000023" izz="0.006096" />
+            </inertial>-->
     </link>
     <link name="${prefix}link_1">
@@ -39,4 +44,8 @@
         </geometry>
       </collision>
+     <!-- <inertial>
+                <mass value="0.0" />
+                <inertia ixx="0.012932" ixy="0.003309" ixz=" -0.000331" iyy="0.018366" iyz="-0.000071" izz="0.019767" />
+            </inertial>-->
     </link>
     <link name="${prefix}link_2">
@@ -54,4 +63,8 @@
         </geometry>
       </collision>
+      <!--<inertial>
+                <mass value="0.0" />
+                <inertia ixx="0.014390" ixy="0.000091" ixz="-0.000323" iyy="0.015120" iyz="-0.001213" izz="0.002053" />
+            </inertial>-->
     </link>
     <link name="${prefix}link_3">
@@ -69,4 +82,8 @@
         </geometry>
       </collision>
+      <!--<inertial>
+               <mass value="0.0" />
+               <inertia ixx="0.001451" ixy="0.000017" ixz="-0.000177" iyy="0.001441" iyz="0.000072" izz="0.001041" />
+           </inertial>-->
     </link>
     <link name="${prefix}link_4">
@@ -84,4 +101,8 @@
         </geometry>
       </collision>
+      <!--<inertial>
+               <mass value="0.0" />
+               <inertia ixx="0.000333" ixy="0.000044" ixz="0.000006" iyy="0.004287" iyz="-0.000000" izz="0.004282" />
+           </inertial>-->
     </link>
     <link name="${prefix}link_5">
@@ -99,4 +120,8 @@
         </geometry>
       </collision>
+      <!--<inertial>
+                <mass value="0.0" />
+                <inertia ixx="0.000088" ixy="-0.000012" ixz="0.000000" iyy="0.000094" iyz="0.000000" izz="0.000118" />
+            </inertial>-->
     </link>
     <link name="${prefix}link_6">
@@ -114,4 +139,8 @@
         </geometry>
       </collision>
+      <!--<inertial>
+                <mass value="0.0" />
+                <inertia ixx="0.000002" ixy="0.000000" ixz="-0.000000" iyy="0.000001" iyz="0.000000" izz="0.000001" />
+            </inertial>-->
     </link>
     <link name="${prefix}ef">
@@ -129,4 +158,8 @@
             </geometry>
           </collision>
+          <!--<inertial>
+                       <mass value="3.0" />
+                       <inertia ixx="0.000127" ixy="0.000000" ixz="0.000052" iyy="0.000194" iyz="0.000003" izz="0.000141" />
+                   </inertial>-->
         </link>
     <!-- joints: main serial chain -->
