Commit message: 2021-4-6 edit inertial tag

File: src/collaborative-robotic-sanding/fanuc_r2000ic_support/urdf/r2000ic165f_macro.xacro (robot description, xacro)
@@ -24,15 +24,75 @@
         </geometry>
       </collision>
-      <!--
+      <inertial>
+               <mass value="10.0" />
+               <origin rpy="0 0 0" xyz="0.0 0.0 0.0" />
+               <inertia ixx="0.002695" ixy="0.000023" ixz="0.000157" iyy="0.004043" iyz="0.000023" izz="0.006096" />
+      </inertial>
+    </link>
+    <link name="${prefix}link_1">
+      <visual>
+        <origin xyz="0 0 0" rpy="0 0 0"/>
+        <geometry>
+          <mesh filename="package://fanuc_r2000ic_support/meshes/r2000ic165f/visual/link_1.stl"/>
+        </geometry>
+        <xacro:material_fanuc_yellow />
+      </visual>
+      <collision>
+        <origin xyz="0 0 0" rpy="0 0 0"/>
+        <geometry>
+          <mesh filename="package://fanuc_r2000ic_support/meshes/r2000ic165f/collision/link_1.stl"/>
+        </geometry>
+      </collision>
+      <inertial>
+                <mass value="0.0" />
+                <origin rpy="0 0 0" xyz="0.0 0.0 0.0" />
+                <inertia ixx="0.012932" ixy="0.003309" ixz=" -0.000331" iyy="0.018366" iyz="-0.000071" izz="0.019767" />
+      </inertial>
+    </link>
+    <link name="${prefix}link_2">
+      <visual>
+        <origin xyz="0 0 0" rpy="0 0 0"/>
+        <geometry>
+          <mesh filename="package://fanuc_r2000ic_support/meshes/r2000ic165f/visual/link_2.stl"/>
+        </geometry>
+        <xacro:material_fanuc_yellow />
+      </visual>
+      <collision>
+        <origin xyz="0 0 0" rpy="0 0 0"/>
+        <geometry>
+          <mesh filename="package://fanuc_r2000ic_support/meshes/r2000ic165f/collision/link_2.stl"/>
+        </geometry>
+      </collision>
+      <inertial>
+                <mass value="0.0" />
+                <origin rpy="0 0 0" xyz="0.0 0.0 0.0" />
+                <inertia ixx="0.014390" ixy="0.000091" ixz="-0.000323" iyy="0.015120" iyz="-0.001213" izz="0.002053" />
+      </inertial>
+    </link>
+    <link name="${prefix}link_3">
+      <visual>
+        <origin xyz="0 0 0" rpy="0 0 0"/>
+        <geometry>
+          <mesh filename="package://fanuc_r2000ic_support/meshes/r2000ic165f/visual/link_3.stl"/>
+        </geometry>
+        <xacro:material_fanuc_yellow />
+      </visual>
+      <collision>
+        <origin xyz="0 0 0" rpy="0 0 0"/>
+        <geometry>
+          <mesh filename="package://fanuc_r2000ic_support/meshes/r2000ic165f/collision/link_3.stl"/>
+        </geometry>
+      </collision>
       <inertial>
                <mass value="0.0" />
-                <inertia ixx="0.002695" ixy="0.000023" ixz="0.000157" iyy="0.004043" iyz="0.000023" izz="0.006096" />
-            </inertial>-->
-    </link>
-    <link name="${prefix}link_1">
-      <visual>
-        <origin xyz="0 0 0" rpy="0 0 0"/>
-        <geometry>
-          <mesh filename="package://fanuc_r2000ic_support/meshes/r2000ic165f/visual/link_1.stl"/>
+               <origin rpy="0 0 0" xyz="0.0 0.0 0.0" />
+               <inertia ixx="0.001451" ixy="0.000017" ixz="-0.000177" iyy="0.001441" iyz="0.000072" izz="0.001041" />
+      </inertial>
+    </link>
+    <link name="${prefix}link_4">
+      <visual>
+        <origin xyz="0 0 0" rpy="0 0 0"/>
+        <geometry>
+          <mesh filename="package://fanuc_r2000ic_support/meshes/r2000ic165f/visual/link_4.stl"/>
         </geometry>
         <xacro:material_fanuc_yellow />
@@ -41,106 +101,52 @@
         <origin xyz="0 0 0" rpy="0 0 0"/>
         <geometry>
-          <mesh filename="package://fanuc_r2000ic_support/meshes/r2000ic165f/collision/link_1.stl"/>
-        </geometry>
-      </collision>
-     <!-- <inertial>
+          <mesh filename="package://fanuc_r2000ic_support/meshes/r2000ic165f/collision/link_4.stl"/>
+        </geometry>
+      </collision>
+      <inertial>
+               <mass value="0.0" />
+               <origin rpy="0 0 0" xyz="0.0 0.0 0.0" />
+               <inertia ixx="0.000333" ixy="0.000044" ixz="0.000006" iyy="0.004287" iyz="-0.000000" izz="0.004282" />
+      </inertial>
+    </link>
+    <link name="${prefix}link_5">
+      <visual>
+        <origin xyz="0 0 0" rpy="0 0 0"/>
+        <geometry>
+          <mesh filename="package://fanuc_r2000ic_support/meshes/r2000ic165f/visual/link_5.stl"/>
+        </geometry>
+        <xacro:material_fanuc_yellow />
+      </visual>
+      <collision>
+        <origin xyz="0 0 0" rpy="0 0 0"/>
+        <geometry>
+          <mesh filename="package://fanuc_r2000ic_support/meshes/r2000ic165f/collision/link_5.stl"/>
+        </geometry>
+      </collision>
+      <inertial>
                 <mass value="0.0" />
-                <inertia ixx="0.012932" ixy="0.003309" ixz=" -0.000331" iyy="0.018366" iyz="-0.000071" izz="0.019767" />
-            </inertial>-->
-    </link>
-    <link name="${prefix}link_2">
-      <visual>
-        <origin xyz="0 0 0" rpy="0 0 0"/>
-        <geometry>
-          <mesh filename="package://fanuc_r2000ic_support/meshes/r2000ic165f/visual/link_2.stl"/>
-        </geometry>
-        <xacro:material_fanuc_yellow />
-      </visual>
-      <collision>
-        <origin xyz="0 0 0" rpy="0 0 0"/>
-        <geometry>
-          <mesh filename="package://fanuc_r2000ic_support/meshes/r2000ic165f/collision/link_2.stl"/>
-        </geometry>
-      </collision>
-      <!--<inertial>
+                <origin rpy="0 0 0" xyz="0.0 0.0 0.0" />
+                <inertia ixx="0.000088" ixy="-0.000012" ixz="0.000000" iyy="0.000094" iyz="0.000000" izz="0.000118" />
+      </inertial>
+    </link>
+    <link name="${prefix}link_6">
+      <visual>
+        <origin xyz="0 0 0" rpy="0 0 0"/>
+        <geometry>
+          <mesh filename="package://fanuc_r2000ic_support/meshes/r2000ic165f/visual/link_6.stl"/>
+        </geometry>
+        <xacro:material_fanuc_black />
+      </visual>
+      <collision>
+        <origin xyz="0 0 0" rpy="0 0 0"/>
+        <geometry>
+          <mesh filename="package://fanuc_r2000ic_support/meshes/r2000ic165f/collision/link_6.stl"/>
+        </geometry>
+      </collision>
+      <inertial>
                 <mass value="0.0" />
-                <inertia ixx="0.014390" ixy="0.000091" ixz="-0.000323" iyy="0.015120" iyz="-0.001213" izz="0.002053" />
-            </inertial>-->
-    </link>
-    <link name="${prefix}link_3">
-      <visual>
-        <origin xyz="0 0 0" rpy="0 0 0"/>
-        <geometry>
-          <mesh filename="package://fanuc_r2000ic_support/meshes/r2000ic165f/visual/link_3.stl"/>
-        </geometry>
-        <xacro:material_fanuc_yellow />
-      </visual>
-      <collision>
-        <origin xyz="0 0 0" rpy="0 0 0"/>
-        <geometry>
-          <mesh filename="package://fanuc_r2000ic_support/meshes/r2000ic165f/collision/link_3.stl"/>
-        </geometry>
-      </collision>
-      <!--<inertial>
-               <mass value="0.0" />
-               <inertia ixx="0.001451" ixy="0.000017" ixz="-0.000177" iyy="0.001441" iyz="0.000072" izz="0.001041" />
-           </inertial>-->
-    </link>
-    <link name="${prefix}link_4">
-      <visual>
-        <origin xyz="0 0 0" rpy="0 0 0"/>
-        <geometry>
-          <mesh filename="package://fanuc_r2000ic_support/meshes/r2000ic165f/visual/link_4.stl"/>
-        </geometry>
-        <xacro:material_fanuc_yellow />
-      </visual>
-      <collision>
-        <origin xyz="0 0 0" rpy="0 0 0"/>
-        <geometry>
-          <mesh filename="package://fanuc_r2000ic_support/meshes/r2000ic165f/collision/link_4.stl"/>
-        </geometry>
-      </collision>
-      <!--<inertial>
-               <mass value="0.0" />
-               <inertia ixx="0.000333" ixy="0.000044" ixz="0.000006" iyy="0.004287" iyz="-0.000000" izz="0.004282" />
-           </inertial>-->
-    </link>
-    <link name="${prefix}link_5">
-      <visual>
-        <origin xyz="0 0 0" rpy="0 0 0"/>
-        <geometry>
-          <mesh filename="package://fanuc_r2000ic_support/meshes/r2000ic165f/visual/link_5.stl"/>
-        </geometry>
-        <xacro:material_fanuc_yellow />
-      </visual>
-      <collision>
-        <origin xyz="0 0 0" rpy="0 0 0"/>
-        <geometry>
-          <mesh filename="package://fanuc_r2000ic_support/meshes/r2000ic165f/collision/link_5.stl"/>
-        </geometry>
-      </collision>
-      <!--<inertial>
-                <mass value="0.0" />
-                <inertia ixx="0.000088" ixy="-0.000012" ixz="0.000000" iyy="0.000094" iyz="0.000000" izz="0.000118" />
-            </inertial>-->
-    </link>
-    <link name="${prefix}link_6">
-      <visual>
-        <origin xyz="0 0 0" rpy="0 0 0"/>
-        <geometry>
-          <mesh filename="package://fanuc_r2000ic_support/meshes/r2000ic165f/visual/link_6.stl"/>
-        </geometry>
-        <xacro:material_fanuc_black />
-      </visual>
-      <collision>
-        <origin xyz="0 0 0" rpy="0 0 0"/>
-        <geometry>
-          <mesh filename="package://fanuc_r2000ic_support/meshes/r2000ic165f/collision/link_6.stl"/>
-        </geometry>
-      </collision>
-      <!--<inertial>
-                <mass value="0.0" />
+                <origin rpy="0 0 0" xyz="0.0 0.0 0.0" />
                 <inertia ixx="0.000002" ixy="0.000000" ixz="-0.000000" iyy="0.000001" iyz="0.000000" izz="0.000001" />
-            </inertial>-->
+      </inertial>
     </link>
     <link name="${prefix}ef">
@@ -158,8 +164,9 @@
             </geometry>
           </collision>
-          <!--<inertial>
+          <inertial>
                        <mass value="3.0" />
+                       <origin rpy="0 0 0" xyz="0.0 0.0 0.0" />
                        <inertia ixx="0.000127" ixy="0.000000" ixz="0.000052" iyy="0.000194" iyz="0.000003" izz="0.000141" />
-                   </inertial>-->
+           </inertial>
         </link>
     <!-- joints: main serial chain -->
@@ -383,5 +390,5 @@
         <selfCollide>true</selfCollide>
     </gazebo>
-    <gazebo reference="gazebo_camera_link">
+<gazebo reference="gazebo_camera_link">
         <sensor type="depth" name="sensor_name">
           <!-- Set always_on only sensor, not on plugin -->

Commit message: 2021-4-6 add joints in ls

File: src/collaborative-robotic-sanding/fanuc_r2000ic_support/urdf/r2000ic165f_macro.xacro (robot description, xacro)
@@ -45,6 +45,6 @@
       </collision>
       <inertial>
-                <mass value="0.0" />
-                <origin rpy="0 0 0" xyz="0.0 0.0 0.0" />
+                <mass value="5.0" />
+                <origin rpy="0 0 0" xyz="0.010863 0.053239 0.523328" />
                 <inertia ixx="0.012932" ixy="0.003309" ixz=" -0.000331" iyy="0.018366" iyz="-0.000071" izz="0.019767" />
       </inertial>
@@ -65,6 +65,6 @@
       </collision>
       <inertial>
-                <mass value="0.0" />
-                <origin rpy="0 0 0" xyz="0.0 0.0 0.0" />
+                <mass value="4.0" />
+                <origin rpy="0 0 0" xyz="-0.001481 0.204359 0.436864" />
                 <inertia ixx="0.014390" ixy="0.000091" ixz="-0.000323" iyy="0.015120" iyz="-0.001213" izz="0.002053" />
       </inertial>
@@ -85,6 +85,6 @@
       </collision>
       <inertial>
-               <mass value="0.0" />
-               <origin rpy="0 0 0" xyz="0.0 0.0 0.0" />
+               <mass value="4.0" />
+               <origin rpy="0 0 0" xyz="0.059293 0.012994 0.109078" />
                <inertia ixx="0.001451" ixy="0.000017" ixz="-0.000177" iyy="0.001441" iyz="0.000072" izz="0.001041" />
       </inertial>
@@ -105,6 +105,6 @@
       </collision>
       <inertial>
-               <mass value="0.0" />
-               <origin rpy="0 0 0" xyz="0.0 0.0 0.0" />
+               <mass value="5.0" />
+               <origin rpy="0 0 0" xyz="0.711733 -0.002537 -0.000643" />
                <inertia ixx="0.000333" ixy="0.000044" ixz="0.000006" iyy="0.004287" iyz="-0.000000" izz="0.004282" />
       </inertial>
@@ -125,6 +125,6 @@
       </collision>
       <inertial>
-                <mass value="0.0" />
-                <origin rpy="0 0 0" xyz="0.0 0.0 0.0" />
+                <mass value="8.0" />
+                <origin rpy="0 0 0" xyz="0.042035 -0.024095 -0.001620" />
                 <inertia ixx="0.000088" ixy="-0.000012" ixz="0.000000" iyy="0.000094" iyz="0.000000" izz="0.000118" />
       </inertial>
@@ -145,6 +145,6 @@
       </collision>
       <inertial>
-                <mass value="0.0" />
-                <origin rpy="0 0 0" xyz="0.0 0.0 0.0" />
+                <mass value="5.0" />
+                <origin rpy="0 0 0" xyz="-0.018677 -0.000000 -0.000002" />
                 <inertia ixx="0.000002" ixy="0.000000" ixz="-0.000000" iyy="0.000001" iyz="0.000000" izz="0.000001" />
       </inertial>

Commit message: 2021-4-16 modify joint 1 line

File: src/collaborative-robotic-sanding/fanuc_r2000ic_support/urdf/r2000ic165f_macro.xacro (robot description, xacro)
@@ -187,5 +187,5 @@
         </link>
     <!-- joints: main serial chain -->
-    <joint name="${prefix}joint_1" type="revolute">
+    <joint name="${prefix}joint_1" type="fixed">
       <origin xyz="0 0 0" rpy="0 0 0"/>
       <parent link="${prefix}base_link"/>
@@ -267,5 +267,5 @@
     </joint>
     <joint name="${prefix}flange-ef" type="fixed">
-          <origin xyz="0 0 0" rpy="${radians(180)} ${radians(-90)} 0" />
+          <origin xyz="0 0 0" rpy="${radians(180)} ${radians(-180)} 0" />
           <parent link="${prefix}tool0" />
           <child link="${prefix}ef" />

Commit message: 2021-4-20 modify scan

File: src/collaborative-robotic-sanding/fanuc_r2000ic_support/urdf/r2000ic165f_macro.xacro (robot description, xacro)
@@ -24,11 +24,9 @@
         </geometry>
       </collision>
-      <!--
       <inertial>
                <mass value="10.0" />
-               <origin rpy="0 0 0" xyz="0.0 0.0 0.0" />
+               <origin rpy="0.002688 0.004043 0.006103" xyz="-0.064613 -0.005314 0.100271" />
                <inertia ixx="0.002695" ixy="0.000023" ixz="0.000157" iyy="0.004043" iyz="0.000023" izz="0.006096" />
       </inertial>
-      -->
     </link>
     <link name="${prefix}link_1">
@@ -46,11 +44,9 @@
         </geometry>
       </collision>
-      <!--
       <inertial>
                 <mass value="5.0" />
-                <origin rpy="0 0 0" xyz="0.010863 0.053239 0.523328" />
+                <origin rpy="0.011358 0.019634 0.020073" xyz="0.010863 0.053239 0.523328" />
                 <inertia ixx="0.012932" ixy="0.003309" ixz=" -0.000331" iyy="0.018366" iyz="-0.000071" izz="0.019767" />
       </inertial>
-      -->
     </link>
     <link name="${prefix}link_2">
@@ -68,11 +64,9 @@
         </geometry>
       </collision>
-      <!--
       <inertial>
                 <mass value="4.0" />
-                <origin rpy="0 0 0" xyz="-0.001481 0.204359 0.436864" />
+                <origin rpy="0.001934 0.014381 0.015249" xyz="-0.001481 0.204359 0.436864" />
                 <inertia ixx="0.014390" ixy="0.000091" ixz="-0.000323" iyy="0.015120" iyz="-0.001213" izz="0.002053" />
       </inertial>
-      -->
     </link>
     <link name="${prefix}link_3">
@@ -90,11 +84,9 @@
         </geometry>
       </collision>
-      <!--
       <inertial>
                <mass value="4.0" />
-               <origin rpy="0 0 0" xyz="0.059293 0.012994 0.109078" />
+               <origin rpy="0.000964 0.001451 0.001518" xyz="0.059293 0.012994 0.109078" />
                <inertia ixx="0.001451" ixy="0.000017" ixz="-0.000177" iyy="0.001441" iyz="0.000072" izz="0.001041" />
       </inertial>
-      -->
     </link>
     <link name="${prefix}link_4">
@@ -112,11 +104,9 @@
         </geometry>
       </collision>
-      <!--
       <inertial>
                <mass value="5.0" />
-               <origin rpy="0 0 0" xyz="0.711733 -0.002537 -0.000643" />
+               <origin rpy="0.000333 0.004282 0.004287" xyz="0.711733 -0.002537 -0.000643" />
                <inertia ixx="0.000333" ixy="0.000044" ixz="0.000006" iyy="0.004287" iyz="-0.000000" izz="0.004282" />
       </inertial>
-      -->
     </link>
     <link name="${prefix}link_5">
@@ -134,11 +124,9 @@
         </geometry>
       </collision>
-      <!--
       <inertial>
                 <mass value="8.0" />
-                <origin rpy="0 0 0" xyz="0.042035 -0.024095 -0.001620" />
+                <origin rpy="0.000078 0.000103 0.000118" xyz="0.042035 -0.024095 -0.001620" />
                 <inertia ixx="0.000088" ixy="-0.000012" ixz="0.000000" iyy="0.000094" iyz="0.000000" izz="0.000118" />
       </inertial>
-      -->
     </link>
     <link name="${prefix}link_6">
@@ -156,11 +144,9 @@
         </geometry>
       </collision>
-      <!--
       <inertial>
                 <mass value="5.0" />
-                <origin rpy="0 0 0" xyz="-0.018677 -0.000000 -0.000002" />
+                <origin rpy="0.000001 0.000001 0.000002" xyz="-0.018677 -0.000000 -0.000002" />
                 <inertia ixx="0.000002" ixy="0.000000" ixz="-0.000000" iyy="0.000001" iyz="0.000000" izz="0.000001" />
       </inertial>
-      -->
     </link>
     <link name="${prefix}ef">
@@ -178,14 +164,12 @@
             </geometry>
           </collision>
-          <!--
           <inertial>
                        <mass value="3.0" />
-                       <origin rpy="0 0 0" xyz="0.0 0.0 0.0" />
+                       <origin rpy="0.000082 0.000185 0.000195" xyz="0.0 0.0 0.0" />
                        <inertia ixx="0.000127" ixy="0.000000" ixz="0.000052" iyy="0.000194" iyz="0.000003" izz="0.000141" />
            </inertial>
-           -->
         </link>
     <!-- joints: main serial chain -->
-    <joint name="${prefix}joint_1" type="fixed">
+    <joint name="${prefix}joint_1" type="revolute">
       <origin xyz="0 0 0" rpy="0 0 0"/>
       <parent link="${prefix}base_link"/>
@@ -289,4 +273,5 @@
         <child link="${prefix}camera_link"/>
     </joint>
+<!--
     <transmission name="joint_1">
         <type>transmission_interface/SimpleTransmission</type>
@@ -406,4 +391,5 @@
         <selfCollide>true</selfCollide>
     </gazebo>
+-->
 <gazebo reference="gazebo_camera_link">
         <sensor type="depth" name="sensor_name">
@@ -459,4 +445,5 @@
           </ros>
           <update_rate>50</update_rate>
+<!--
           <joint_name>${prefix}joint_1</joint_name>
           <joint_name>${prefix}joint_2</joint_name>
@@ -465,4 +452,5 @@
           <joint_name>${prefix}joint_5</joint_name>
           <joint_name>${prefix}joint_6</joint_name>
+-->
         </plugin>
         <plugin name='crs_gazebo_plugins_joint_pose_trajectory' filename='libcrs_gazebo_plugins_joint_pose_trajectory.so'>

Commit message: 2021-5-13 add urdf

File: src/collaborative-robotic-sanding/fanuc_r2000ic_support/urdf/r2000ic165f_macro.xacro (robot description, xacro)
@@ -255,6 +255,6 @@
           <child link="${prefix}ef" />
         </joint>
-<link name="${prefix}tcp" />
-<joint name="${prefix}tcp_ef" type="fixed">
+    <link name="${prefix}tcp" />
+    <joint name="${prefix}tcp_ef" type="fixed">
        <origin xyz="-0.204433413 -7.32E-04 0.333181177" rpy="5.53832e-13 -0.785398 0"/>
       <parent link="${prefix}ef" />

Commit message: 2021-6-17 modify trajectory

File: src/collaborative-robotic-sanding/fanuc_r2000ic_support/urdf/r2000ic165f_macro.xacro (robot description, xacro)
@@ -154,5 +154,6 @@
             <origin xyz="0 0 0" rpy="0 0 0"/>
             <geometry>
-              <mesh filename="package://fanuc_r2000ic_support/meshes/r2000ic165f/visual/ef.stl"/>
+            <!--scale="0.001 0.001 0.001"-->
+              <mesh filename="package://fanuc_r2000ic_support/meshes/r2000ic165f/visual/ef.stl" />
             </geometry>
             <xacro:material_fanuc_yellow />
@@ -161,5 +162,5 @@
             <origin xyz="0 0 0" rpy="0 0 0"/>
             <geometry>
-              <mesh filename="package://fanuc_r2000ic_support/meshes/r2000ic165f/collision/ef.stl"/>
+              <mesh filename="package://fanuc_r2000ic_support/meshes/r2000ic165f/collision/ef.stl" />
             </geometry>
           </collision>
@@ -251,5 +252,7 @@
     </joint>
     <joint name="${prefix}flange-ef" type="fixed">
-          <origin xyz="0 0 0" rpy="${radians(180)} ${radians(-90)} 0" />
+<!--    <origin xyz="0 0 0" rpy="${radians(180)} ${radians(-90)} 0" />-->
+     <origin xyz="0 0 0" rpy="${radians(180)} ${radians(-90)} 0" />
+<!--         <origin xyz="-0.02 0.25 -0.3" rpy="${radians(157)} ${radians(-80)} ${radians(12)}" />-->
           <parent link="${prefix}link_6" />
           <child link="${prefix}ef" />

Commit message: 2021-6-21 xiaopeng modify bath p

File: src/collaborative-robotic-sanding/fanuc_r2000ic_support/urdf/r2000ic165f_macro.xacro (robot description, xacro)
@@ -262,4 +262,6 @@
     <!--  <origin xyz="-0.204433413 -7.32E-04 0.333181177" rpy="5.53832e-13 -0.785398 0"/>-->
       <origin xyz="-0.2303 0.1296 0.3799" rpy="${radians(23.9)} ${radians(-38.2)} ${radians(-65.3)}" />
+<!--      <origin xyz="-0.2488 0.1457 0.3941" rpy="${radians(141.6)} ${radians(-23.5)} ${radians(32.3)}" />-->
+      <origin xyz="-0.2488 0.1457 0.3941" rpy="${radians(23.9)} ${radians(-38.2)} ${radians(-65.3)}" />
       <parent link="${prefix}ef" />
       <child link="${prefix}tcp" />
