Commit message: add ef.stl

File: src/collaborative-robotic-sanding/fanuc_r2000ic_support/urdf/r2000ic165f.urdf (robot description, URDF)
Before this commit: robot fanuc_r2000ic165f, 11 links, 10 joints
Links:
- removed link part_link
- added link camera_link
- added link camera_link_optical
- added link gazebo_camera_link
Joints:
- removed joint world_part_link
- added joint camera_link_joint: type fixed, parent camera_link_optical, child camera_link, origin xyz=0.0 0.0 0.0 rpy=1.57 -1.57 0
- added joint camera_optical_joint: type fixed, parent link_6, child camera_link_optical, origin xyz=-0.021 0.0797 0.06525 rpy=-0.7854 0 0
- added joint gazebo_camera_joint: type fixed, parent camera_link_optical, child gazebo_camera_link, origin xyz=0.0 0.0 0.0 rpy=1.57 -1.57 0.0

File: src/collaborative-robotic-sanding/fanuc_r2000ic_support/urdf/r2000ic165f_macro.xacro (robot description, xacro)
@@ -158,4 +158,5 @@
       <limit lower="${radians(-360)}" upper="${radians(360)}" effort="0" velocity="${radians(260)}"/>
     </joint>
+<!--
 <link name="part_link">
   <visual>
@@ -173,5 +174,5 @@
       <child link="part_link" />
       <origin rpy="0 0 0" xyz="1.4 -0.4 0.6" />
-  </joint>
+  </joint>-->
     <!-- ROS-Industrial 'base' frame: base_link to Fanuc World Coordinates transform -->
     <link name="${prefix}base" />
@@ -197,5 +198,5 @@
 <transmission name="joint_1">
     <type>transmission_interface/SimpleTransmission</type>
-    <joint name="${prefix}joint_1">
+    <joint name="joint_1">
         <hardwareInterface>hardware_interface/EffortJointInterface</hardwareInterface>
     </joint>
@@ -205,44 +206,44 @@
     </actuator>
 </transmission>
-<gazebo reference="${prefix}base_link">
-    <selfCollide>true</selfCollide>
-</gazebo>
-<gazebo reference="${prefix}link_1">
-    <selfCollide>true</selfCollide>
-</gazebo>
-<gazebo reference="${prefix}link_2">
-    <selfCollide>true</selfCollide>
-</gazebo>
-<gazebo reference="${prefix}link_3">
-    <selfCollide>true</selfCollide>
-</gazebo>
-<gazebo reference="${prefix}link_4">
-    <selfCollide>true</selfCollide>
-</gazebo>
-<gazebo reference="${prefix}link_5">
-    <selfCollide>true</selfCollide>
-</gazebo>
-<gazebo reference="${prefix}link_6">
-    <selfCollide>true</selfCollide>
-</gazebo>
-<gazebo reference="${prefix}joint_1">
-    <selfCollide>true</selfCollide>
-</gazebo>
-<gazebo reference="${prefix}joint_2">
-    <selfCollide>true</selfCollide>
-</gazebo>
-<gazebo reference="${prefix}joint_3">
-    <selfCollide>true</selfCollide>
-</gazebo>
-<gazebo reference="${prefix}base">
-    <selfCollide>true</selfCollide>
-</gazebo>
-<gazebo reference="${prefix}flange">
-    <selfCollide>true</selfCollide>
-</gazebo>
-<gazebo reference="${prefix}tool0">
-    <selfCollide>true</selfCollide>
-</gazebo>
-<gazebo reference="${prefix}gazebo_camera_link">
+<gazebo reference="base_link">
+    <selfCollide>true</selfCollide>
+</gazebo>
+<gazebo reference="link_1">
+    <selfCollide>true</selfCollide>
+</gazebo>
+<gazebo reference="link_2">
+    <selfCollide>true</selfCollide>
+</gazebo>
+<gazebo reference="link_3">
+    <selfCollide>true</selfCollide>
+</gazebo>
+<gazebo reference="link_4">
+    <selfCollide>true</selfCollide>
+</gazebo>
+<gazebo reference="link_5">
+    <selfCollide>true</selfCollide>
+</gazebo>
+<gazebo reference="link_6">
+    <selfCollide>true</selfCollide>
+</gazebo>
+<gazebo reference="joint_1">
+    <selfCollide>true</selfCollide>
+</gazebo>
+<gazebo reference="joint_2">
+    <selfCollide>true</selfCollide>
+</gazebo>
+<gazebo reference="joint_3">
+    <selfCollide>true</selfCollide>
+</gazebo>
+<gazebo reference="base">
+    <selfCollide>true</selfCollide>
+</gazebo>
+<gazebo reference="flange">
+    <selfCollide>true</selfCollide>
+</gazebo>
+<gazebo reference="tool0">
+    <selfCollide>true</selfCollide>
+</gazebo>
+<gazebo reference="gazebo_camera_link">
     <sensor type="depth" name="sensor_name">
       <!-- Set always_on only sensor, not on plugin -->
@@ -297,15 +298,15 @@
       </ros>
       <update_rate>50</update_rate>
-      <joint_name>${prefix}joint_1</joint_name>
-      <joint_name>${prefix}joint_2</joint_name>
-      <joint_name>${prefix}joint_3</joint_name>
-      <joint_name>${prefix}joint_4</joint_name>
-      <joint_name>${prefix}joint_5</joint_name>
-      <joint_name>${prefix}joint_6</joint_name>
+      <joint_name>joint_1</joint_name>
+      <joint_name>joint_2</joint_name>
+      <joint_name>joint_3</joint_name>
+      <joint_name>joint_4</joint_name>
+      <joint_name>joint_5</joint_name>
+      <joint_name>joint_6</joint_name>
     </plugin>
     <plugin name='crs_gazebo_plugins_joint_pose_trajectory' filename='libcrs_gazebo_plugins_joint_pose_trajectory.so'>
         <ros>
           <namespace>sim</namespace>
-          <argument>follow_joint_trajectory:=${prefix}follow_joint_trajectory</argument>
+          <argument>follow_joint_trajectory:=follow_joint_trajectory</argument>
         </ros>
         <update_rate>20</update_rate>

Commit message: 3-16 modify fanuc robot

File: src/collaborative-robotic-sanding/fanuc_r2000ic_support/urdf/r2000ic165f.urdf (robot description, URDF)
Before this commit: robot fanuc_r2000ic165f, 13 links, 12 joints
Links:
- added link ef; collision mesh filename=package://fanuc_r2000ic_support/meshes/r2000ic165f/collisio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; visual mesh filename=package://fanuc_r2000ic_support/meshes/r2000ic165f/visual/e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
Joints:
- added joint flange-ef: type fixed, parent flange, child ef, origin xyz=0 0 0 rpy=3.14159265359 -1.57079632679 0

File: src/collaborative-robotic-sanding/fanuc_r2000ic_support/urdf/r2000ic165f_macro.xacro (robot description, xacro)
@@ -115,4 +115,19 @@
       </collision>
     </link>
+    <link name="${prefix}ef">
+          <visual>
+            <origin xyz="0 0 0" rpy="0 0 0"/>
+            <geometry>
+              <mesh filename="package://fanuc_r2000ic_support/meshes/r2000ic165f/visual/ef.stl"/>
+            </geometry>
+            <xacro:material_fanuc_yellow />
+          </visual>
+          <collision>
+            <origin xyz="0 0 0" rpy="0 0 0"/>
+            <geometry>
+              <mesh filename="package://fanuc_r2000ic_support/meshes/r2000ic165f/collision/ef.stl"/>
+            </geometry>
+          </collision>
+        </link>
     <!-- joints: main serial chain -->
     <joint name="${prefix}joint_1" type="revolute">
@@ -196,4 +211,9 @@
       <child link="${prefix}tool0" />
     </joint>
+    <joint name="${prefix}flange-ef" type="fixed">
+          <origin xyz="0 0 0" rpy="${radians(180)} ${radians(-90)} 0" />
+          <parent link="${prefix}flange" />
+          <child link="${prefix}ef" />
+        </joint>
 <transmission name="joint_1">
     <type>transmission_interface/SimpleTransmission</type>

Commit message: 2021-4-28 xiao modify urdf srdf configuration

File: src/collaborative-robotic-sanding/fanuc_r2000ic_support/urdf/r2000ic165f.urdf (robot description, URDF)
Before this commit: robot fanuc_r2000ic165f, 14 links, 13 joints
Links:
- added link world
- link base_link: mass None -> 10.0
- link ef: mass None -> 3.0
- link gazebo_camera_link: mass None -> 1e-5; geometry collision box size=0.1 0.1 0.1; visual box size=0.1 0.1 0.1
- link link_1: mass None -> 5.0
- link link_2: mass None -> 4.0
- link link_3: mass None -> 4.0
- link link_4: mass None -> 5.0
- link link_5: mass None -> 8.0
- link link_6: mass None -> 5.0
Joints:
- added joint world_base_link: type fixed, parent world, child base_link, origin xyz=-2.5 0 0 rpy=0 0 0
- joint camera_optical_joint: origin xyz=-0.021 0.0797 0.06525 rpy=-0.7854 0 0 -> xyz=0.1 0 0.2 rpy=0 0 0; parent link_6 -> ef
- joint flange-ef: origin xyz=0 0 0 rpy=3.14159265359 -1.57079632679 0 -> xyz=0 0 0 rpy=3.141592653589793 -3.141592653589793 0; parent flange -> tool0
- joint flange-tool0: origin xyz=0 0 0 rpy=0 1.57079632679 0 -> xyz=0 0 0 rpy=0 1.5707963267948966 0; parent flange -> link_6
- joint gazebo_camera_joint: origin xyz=0.0 0.0 0.0 rpy=1.57 -1.57 0.0 -> xyz=0.0 0.0 0.0 rpy=0 -1.57 0
- joint joint_1: limit lower=-3.22885911619 upper=3.22885911619 effort=0 velocity=2.26892802759 -> lower=-3.2288591161895095 upper=3.2288591161895095 effort=0 velocity=2.2689280275926285
- joint joint_2: limit lower=-1.0471975512 upper=1.32645023152 effort=0 velocity=2.00712863979 -> lower=-1.0471975511965976 upper=1.3264502315156905 effort=0 velocity=2.007128639793479
- joint joint_3: limit lower=-2.30383461263 upper=3.14159265359 effort=0 velocity=2.18166156499 -> lower=-2.303834612632515 upper=3.141592653589793 effort=0 velocity=2.181661564992912
- joint joint_4: limit lower=-6.28318530718 upper=6.28318530718 effort=0 velocity=3.14159265359 -> lower=-6.283185307179586 upper=6.283185307179586 effort=0 velocity=3.141592653589793
- joint joint_5: limit lower=-2.18166156499 upper=2.18166156499 effort=0 velocity=3.14159265359 -> lower=-2.181661564992912 upper=2.181661564992912 effort=0 velocity=3.141592653589793
- joint joint_6: limit lower=-6.28318530718 upper=6.28318530718 effort=0 velocity=4.53785605519 -> lower=-6.283185307179586 upper=6.283185307179586 effort=0 velocity=4.537856055185257

File: src/collaborative-robotic-sanding/fanuc_r2000ic_support/urdf/r2000ic165f_macro.xacro (robot description, xacro)
@@ -1,5 +1,5 @@
 <?xml version="1.0"?>
 <robot xmlns:xacro="http://wiki.ros.org/xacro">
-  <xacro:include filename="$(find fanuc_resources)/urdf/common_materials.xacro"/>
+  <xacro:include filename="$(find fanuc_resources)/urdf/common_materials.xacro"  />
   <xacro:macro name="fanuc_r2000ic165f" params="prefix">
     <!-- links: main serial chain -->
@@ -247,5 +247,5 @@
     <joint name="${prefix}flange-tool0" type="fixed">
       <origin xyz="0 0 0" rpy="0 ${radians(90)} 0" />
-      <parent link="${prefix}flange" />
+      <parent link="${prefix}link_6" />
       <child link="${prefix}tool0" />
     </joint>
@@ -255,13 +255,33 @@
           <child link="${prefix}ef" />
         </joint>
-    <link name="${prefix}gazebo_camera_link" />
+    <link name="${prefix}gazebo_camera_link" >
+    <collision>
+      <origin xyz="0 0 0" rpy="0 0 0"/>
+      <geometry>
+        <box size="0.1 0.1 0.1"/>
+      </geometry>
+    </collision>
+    <visual>
+      <origin xyz="0 0 0" rpy="0 0 0"/>
+      <geometry>
+         <box size="0.1 0.1 0.1"/>
+      </geometry>
+      <xacro:material_fanuc_yellow />
+    </visual>
+    <inertial>
+      <mass value="1e-5" />
+      <origin xyz="0 0 0" rpy="0 0 0"/>
+      <inertia ixx="1e-6" ixy="0" ixz="0" iyy="1e-6" iyz="0" izz="1e-6" />
+    </inertial>
+    </link>
     <joint name="${prefix}gazebo_camera_joint" type="fixed">
-        <origin xyz="0.0 0.0 0.0" rpy="1.57 -1.57 0.0"/>
+        <origin xyz="0.0 0.0 0.0" rpy="0 -1.57 0"/>
         <parent link="${prefix}camera_link_optical"/>
         <child link="${prefix}gazebo_camera_link"/>
     </joint>
-    <link name="${prefix}camera_link_optical" />
+    <link name="${prefix}camera_link_optical">
+    </link>
     <joint name="${prefix}camera_optical_joint" type="fixed">
-        <origin xyz="-0.021 0.0797 0.06525" rpy="-0.7854 0 0"/>
+        <origin xyz="0.1 0 0.2" rpy="0 0 0"/>
         <parent link="${prefix}ef"/>
         <child link="${prefix}camera_link_optical"/>
@@ -273,6 +293,5 @@
         <child link="${prefix}camera_link"/>
     </joint>
-<!--
-    <transmission name="joint_1">
+    <transmission name="trans_joint_1">
         <type>transmission_interface/SimpleTransmission</type>
         <joint name="${prefix}joint_1">
@@ -284,5 +303,5 @@
         </actuator>
     </transmission>
-<transmission name="joint_2">
+<transmission name="trans_joint_2">
     <type>transmission_interface/SimpleTransmission</type>
     <joint name="${prefix}joint_2">
@@ -294,5 +313,5 @@
     </actuator>
 </transmission>
-<transmission name="joint_3">
+<transmission name="trans_joint_3">
     <type>transmission_interface/SimpleTransmission</type>
     <joint name="${prefix}joint_3">
@@ -304,5 +323,5 @@
     </actuator>
 </transmission>
-<transmission name="joint_4">
+<transmission name="trans_joint_4">
     <type>transmission_interface/SimpleTransmission</type>
     <joint name="${prefix}joint_4">
@@ -314,5 +333,5 @@
     </actuator>
 </transmission>
-<transmission name="joint_5">
+<transmission name="trans_joint_5">
     <type>transmission_interface/SimpleTransmission</type>
     <joint name="${prefix}joint_5">
@@ -324,5 +343,5 @@
     </actuator>
 </transmission>
-<transmission name="joint_6">
+<transmission name="trans_joint_6">
     <type>transmission_interface/SimpleTransmission</type>
     <joint name="${prefix}joint_6">
@@ -358,39 +377,49 @@
         <selfCollide>true</selfCollide>
     </gazebo>
-    <gazebo reference="${prefix}joint_1">
-        <selfCollide>true</selfCollide>
-    </gazebo>
-    <gazebo reference="${prefix}joint_2">
-        <selfCollide>true</selfCollide>
-    </gazebo>
-    <gazebo reference="${prefix}joint_3">
-        <selfCollide>true</selfCollide>
-    </gazebo>
-    <gazebo reference="${prefix}joint_4">
-        <selfCollide>true</selfCollide>
-    </gazebo>
-    <gazebo reference="${prefix}joint_5">
-        <selfCollide>true</selfCollide>
-    </gazebo>
-    <gazebo reference="${prefix}joint_6">
-        <selfCollide>true</selfCollide>
-    </gazebo>
-    <gazebo reference="${prefix}flange-ef">
-        <selfCollide>true</selfCollide>
-    </gazebo>
     <gazebo reference="${prefix}tool0">
         <selfCollide>true</selfCollide>
     </gazebo>
-    <gazebo reference="${prefix}base">
-        <selfCollide>true</selfCollide>
-    </gazebo>
     <gazebo reference="${prefix}flange">
         <selfCollide>true</selfCollide>
     </gazebo>
-    <gazebo reference="tool0">
-        <selfCollide>true</selfCollide>
-    </gazebo>
+<!-- camera
+ <gazebo reference="camera_link">
+   <sensor type="camera" name="camera1">
+     <update_rate>30.0</update_rate>
+     <camera name="head">
+       <horizontal_fov>1.3962634</horizontal_fov>
+       <image>
+         <width>800</width>
+         <height>800</height>
+         <format>R8G8B8</format>
+       </image>
+       <clip>
+         <near>0.02</near>
+         <far>300</far>
+       </clip>
+       <noise>
+         <type>gaussian</type>
+         <mean>0.0</mean>
+         <stddev>0.007</stddev>
+       </noise>
+     </camera>
+     <plugin name="camera_controller" filename="libgazebo_ros_camera.so">
+       <alwaysOn>true</alwaysOn>
+       <updateRate>0.0</updateRate>
+       <cameraName>rrbot/camera1</cameraName>
+       <imageTopicName>image_raw</imageTopicName>
+       <cameraInfoTopicName>camera_info</cameraInfoTopicName>
+       <frameName>camera_link</frameName>
+       <hackBaseline>0.07</hackBaseline>
+       <distortionK1>0.0</distortionK1>
+       <distortionK2>0.0</distortionK2>
+       <distortionK3>0.0</distortionK3>
+       <distortionT1>0.0</distortionT1>
+       <distortionT2>0.0</distortionT2>
+     </plugin>
+   </sensor>
+ </gazebo>
 -->
-<gazebo reference="gazebo_camera_link">
+<gazebo reference="${prefix}gazebo_camera_link">
         <sensor type="depth" name="sensor_name">
           <!-- Set always_on only sensor, not on plugin -->
@@ -445,5 +474,4 @@
           </ros>
           <update_rate>50</update_rate>
-<!--
           <joint_name>${prefix}joint_1</joint_name>
           <joint_name>${prefix}joint_2</joint_name>
@@ -452,5 +480,4 @@
           <joint_name>${prefix}joint_5</joint_name>
           <joint_name>${prefix}joint_6</joint_name>
--->
         </plugin>
         <plugin name='crs_gazebo_plugins_joint_pose_trajectory' filename='libcrs_gazebo_plugins_joint_pose_trajectory.so'>

Commit message: 2021-5-13 modify config add tcp in urdf

File: src/collaborative-robotic-sanding/fanuc_r2000ic_support/urdf/r2000ic165f.urdf (robot description, URDF)
Before this commit: robot crs, 15 links, 14 joints
Links:
- added link tcp
Joints:
- added joint tcp_ef: type fixed, parent ef, child tcp, origin xyz=-0.204433413 -7.32E-04 0.333181177 rpy=5.53832e-13 -0.785398 0
- joint gazebo_camera_joint: origin xyz=0.0 0.0 0.0 rpy=0 -1.57 0 -> xyz=0.0 0.0 0.0 rpy=1.57 -1.57 0

File: src/collaborative-robotic-sanding/fanuc_r2000ic_support/urdf/r2000ic165f_macro.xacro (robot description, xacro)
@@ -255,4 +255,10 @@
           <child link="${prefix}ef" />
         </joint>
+<link name="${prefix}tcp" />
+<joint name="${prefix}tcp_ef" type="fixed">
+       <origin xyz="-0.204433413 -7.32E-04 0.333181177" rpy="5.53832e-13 -0.785398 0"/>
+      <parent link="${prefix}ef" />
+      <child link="${prefix}tcp" />
+    </joint>
     <link name="${prefix}gazebo_camera_link" >
     <collision>
@@ -276,5 +282,5 @@
     </link>
     <joint name="${prefix}gazebo_camera_joint" type="fixed">
-        <origin xyz="0.0 0.0 0.0" rpy="0 -1.57 0"/>
+        <origin xyz="0.0 0.0 0.0" rpy="1.57 -1.57 0"/>
         <parent link="${prefix}camera_link_optical"/>
         <child link="${prefix}gazebo_camera_link"/>

Commit message: 2021-6-4 xiaopeng modify trajectory

File: src/collaborative-robotic-sanding/fanuc_r2000ic_support/urdf/r2000ic165f.urdf (robot description, URDF)
Before this commit: robot crs, 16 links, 15 joints
Joints:
- joint flange-ef: origin xyz=0 0 0 rpy=3.141592653589793 -3.141592653589793 0 -> xyz=0 0 0 rpy=3.141592653589793 -1.5707963267948966 0; parent tool0 -> link_6

File: src/collaborative-robotic-sanding/fanuc_r2000ic_support/urdf/r2000ic165f_macro.xacro (robot description, xacro)
@@ -251,6 +251,6 @@
     </joint>
     <joint name="${prefix}flange-ef" type="fixed">
-          <origin xyz="0 0 0" rpy="${radians(180)} ${radians(-180)} 0" />
-          <parent link="${prefix}tool0" />
+          <origin xyz="0 0 0" rpy="${radians(180)} ${radians(-90)} 0" />
+          <parent link="${prefix}link_6" />
           <child link="${prefix}ef" />
         </joint>

Commit message: 2021-6-16 xiaopeng modify tcp

File: src/collaborative-robotic-sanding/fanuc_r2000ic_support/urdf/r2000ic165f.urdf (robot description, URDF)
Before this commit: robot crs, 16 links, 15 joints
Joints:
- joint tcp_ef: origin xyz=-0.204433413 -7.32E-04 0.333181177 rpy=5.53832e-13 -0.785398 0 -> xyz=-0.2303 0.1296 0.3799 rpy=0.41713369122664473 -0.6667157742618339 -1.1397000015522971

File: src/collaborative-robotic-sanding/fanuc_r2000ic_support/urdf/r2000ic165f_macro.xacro (robot description, xacro)
@@ -257,5 +257,6 @@
     <link name="${prefix}tcp" />
     <joint name="${prefix}tcp_ef" type="fixed">
-       <origin xyz="-0.204433413 -7.32E-04 0.333181177" rpy="5.53832e-13 -0.785398 0"/>
+    <!--  <origin xyz="-0.204433413 -7.32E-04 0.333181177" rpy="5.53832e-13 -0.785398 0"/>-->
+      <origin xyz="-0.2303 0.1296 0.3799" rpy="${radians(23.9)} ${radians(-38.2)} ${radians(-65.3)}" />
       <parent link="${prefix}ef" />
       <child link="${prefix}tcp" />

Commit message: 2021-6-22 xiaopeng test tw

File: src/collaborative-robotic-sanding/fanuc_r2000ic_support/urdf/r2000ic165f.urdf (robot description, URDF)
Before this commit: robot crs, 16 links, 15 joints
Joints:
- joint tcp_ef: origin xyz=-0.2303 0.1296 0.3799 rpy=0.41713369122664473 -0.6667157742618339 -1.1397000015522971 -> xyz=-0.3301 0.006 0.4428 rpy=0.5113814708343386 -0.630063859969953 -0.7696902001294994

File: src/collaborative-robotic-sanding/fanuc_r2000ic_support/urdf/r2000ic165f_macro.xacro (robot description, xacro)
@@ -261,7 +261,7 @@
     <joint name="${prefix}tcp_ef" type="fixed">
     <!--  <origin xyz="-0.204433413 -7.32E-04 0.333181177" rpy="5.53832e-13 -0.785398 0"/>-->
-      <origin xyz="-0.2303 0.1296 0.3799" rpy="${radians(23.9)} ${radians(-38.2)} ${radians(-65.3)}" />
+<!--      <origin xyz="-0.2303 0.1296 0.3799" rpy="${radians(23.9)} ${radians(-38.2)} ${radians(-65.3)}" />-->
 <!--      <origin xyz="-0.2488 0.1457 0.3941" rpy="${radians(141.6)} ${radians(-23.5)} ${radians(32.3)}" />-->
-      <origin xyz="-0.2488 0.1457 0.3941" rpy="${radians(23.9)} ${radians(-38.2)} ${radians(-65.3)}" />
+      <origin xyz="-0.3301 0.006 0.4428" rpy="${radians(29.3)} ${radians(-36.1)} ${radians(-44.1)}" />
       <parent link="${prefix}ef" />
       <child link="${prefix}tcp" />
