Commit message: 2021-4-2

File: src/collaborative-robotic-sanding/crs_support/urdf/crs.urdf.xacro (robot description, xacro)
@@ -562,5 +562,5 @@
         <selfCollide>true</selfCollide>
     </gazebo>
-    <gazebo reference="${prefix}gazebo_camera_link">
+<gazebo reference="${prefix}gazebo_camera_link">
         <sensor type="depth" name="sensor_name">
           <!-- Set always_on only sensor, not on plugin -->

File: src/collaborative-robotic-sanding/fanuc_r2000ic_support/urdf/r2000ic165f_macro.xacro (robot description, xacro)
@@ -245,5 +245,5 @@
     <joint name="${prefix}flange-ef" type="fixed">
           <origin xyz="0 0 0" rpy="${radians(180)} ${radians(-90)} 0" />
-          <parent link="${prefix}flange" />
+          <parent link="${prefix}tool0" />
           <child link="${prefix}ef" />
         </joint>
